File: hardware/cart.kicad_sch (KiCad schematic)
At the start: 9 parts, among them J2 debug-power, P1 edge connector, U1 74LVC138, U2 1.5A @ 3.3V

Commit message: Dummy change to test schematic PDF update in PRs
Other:
- title: Kinetoscope Cartridge Connector -> Kinetoscope Cartridge Connector zzz
Changed lines of the file:
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@@
 	(paper "A4")
 	(title_block
-		(title "Kinetoscope Cartridge Connector")
+		(title "Kinetoscope Cartridge Connector zzz")
 	)
 	(junction
