File: hardware/kinetoscope-header-internal.kicad_sch (KiCad schematic)
At the start: 3 parts

Commit message: Update header part numbers
SSW pins are incompatible with other headers.  SSQ should be better.  (Yet to confirm.)
Parts:
- J1: Mouser Part Number 200-SSW12602TD -> 200-SSQ12603TD; Part Number SSW-126-02-T-D -> SSQ-126-03-T-D
- J2: Mouser Part Number 200-SSW12102TD -> 200-SSQ12103TD; Part Number SSW-121-02-T-D -> SSQ-121-03-T-D
Changed lines of the file:
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@@
 			)
 		)
-		(property "Mouser Part Number" "200-SSW12102TD"
+		(property "Mouser Part Number" "200-SSQ12103TD"
 			(at 204.47 41.91 0)
 			(effects
@@
 			)
 		)
-		(property "Part Number" "SSW-121-02-T-D"
+		(property "Part Number" "SSQ-121-03-T-D"
 			(at 204.47 41.91 0)
 			(effects
@@
 			)
 		)
-		(property "Mouser Part Number" "200-SSW12602TD"
+		(property "Mouser Part Number" "200-SSQ12603TD"
 			(at 62.23 34.29 0)
 			(effects
@@
 			)
 		)
-		(property "Part Number" "SSW-126-02-T-D"
+		(property "Part Number" "SSQ-126-03-T-D"
 			(at 62.23 34.29 0)
 			(effects

Commit message: Drop Samtec headers
They do not connect well.  I need more reliable stacking headers.
Parts:
- J1: JLCPCB Part Number C3323945 -> (none); Mouser Part Number 200-SSQ12603TD -> (none); Part Number SSQ-126-03-T-D -> (none)
- J2: JLCPCB Part Number C3324002 -> (none); Mouser Part Number 200-SSQ12103TD -> (none); Part Number SSQ-121-03-T-D -> (none)
Changed lines of the file:
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@@
 			)
 		)
-		(property "JLCPCB Part Number" "C3324002"
+		(property "JLCPCB Part Number" ""
 			(at 204.47 41.91 0)
 			(effects
@@
 			)
 		)
-		(property "Mouser Part Number" "200-SSQ12103TD"
+		(property "Mouser Part Number" ""
 			(at 204.47 41.91 0)
 			(effects
@@
 			)
 		)
-		(property "Part Number" "SSQ-121-03-T-D"
+		(property "Part Number" ""
 			(at 204.47 41.91 0)
 			(effects
@@
 			)
 		)
-		(property "JLCPCB Part Number" "C3323945"
+		(property "JLCPCB Part Number" ""
 			(at 62.23 34.29 0)
 			(effects
@@
 			)
 		)
-		(property "Mouser Part Number" "200-SSQ12603TD"
+		(property "Mouser Part Number" ""
 			(at 62.23 34.29 0)
 			(effects
@@
 			)
 		)
-		(property "Part Number" "SSQ-126-03-T-D"
+		(property "Part Number" ""
 			(at 62.23 34.29 0)
 			(effects
