File: hardware/unified.kicad_sch (KiCad schematic)
At the start: 0 parts

Commit message: Layout for unified PCB
Manual routing of ground vias, decoupling caps, and regulator
Other:
- title: (none) -> Kinetoscope unified PCB
Changed lines of the file:
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@@
 	(generator_version "9.0")
 	(paper "A4")
+	(title_block
+		(title "Kinetoscope unified PCB")
+	)
 	(wire
 		(pts
